Commit message: Changes by Julian (TFG UAL 2019)

File: schunk_description/urdf/lwa4p/lwa4p.gazebo.xacro (robot description, xacro)
@@ -37,4 +37,19 @@
       <material value="Schunk/LightGrey" />
     </gazebo>
+    <gazebo reference="${name}_gripper_link">
+      <gravity>true</gravity>
+      <self_collide>false</self_collide>
+      <material value="Schunk/Blue" />
+    </gazebo>
+    <gazebo reference="${name}_finger1_link">
+      <gravity>true</gravity>
+      <self_collide>false</self_collide>
+      <material value="Schunk/LightGrey" />
+    </gazebo>
+    <gazebo reference="${name}_finger2_link">
+      <gravity>true</gravity>
+      <self_collide>false</self_collide>
+      <material value="Schunk/LightGrey" />
+    </gazebo>
   </xacro:macro>
 </robot>

File: schunk_description/urdf/lwa4p/lwa4p.urdf.xacro (robot description, xacro)
@@ -55,6 +55,5 @@
     </joint>
     <link name="${name}_1_link">
-      <xacro:default_inertial/>
-<!--
+      <!--xacro:default_inertial/-->
       <inertial>
         <origin xyz="0 0 0" rpy="0 0 0" />
@@ -62,5 +61,4 @@
         <inertia ixx="0.01" ixy="0" ixz="0" iyy="0.01" iyz="0" izz="0.01" />
       </inertial>
--->
       <visual>
         <origin xyz="0 0 0" rpy="0 0 0" />
@@ -87,6 +85,5 @@
     </joint>
     <link name="${name}_2_link">
-      <xacro:default_inertial/>
-<!--
+      <!--xacro:default_inertial/-->
       <inertial>
         <origin xyz="0 0 0" rpy="0 0 0"/>
@@ -94,5 +91,4 @@
         <inertia ixx="0.03" ixy="0" ixz="0" iyy="0.03" iyz="0" izz="0.03" />
       </inertial>
--->
       <visual>
         <origin xyz="0 0 0" rpy="0 0 0" />
@@ -119,6 +115,5 @@
     </joint>
     <link name="${name}_3_link">
-      <xacro:default_inertial/>
-<!--
+      <!--xacro:default_inertial/-->
       <inertial>
         <origin xyz="0 0 0" rpy="0 0 0"/>
@@ -126,5 +121,4 @@
         <inertia ixx="0.03" ixy="0" ixz="0" iyy="0.03" iyz="0" izz="0.03" />
       </inertial>
--->
       <visual>
         <origin xyz="0 0 0" rpy="0 0 0" />
@@ -151,6 +145,5 @@
     </joint>
     <link name="${name}_4_link">
-      <xacro:default_inertial/>
-<!--
+      <!--xacro:default_inertial/-->
       <inertial>
         <origin xyz="0 0 0" rpy="0 0 0"/>
@@ -158,5 +151,4 @@
         <inertia ixx="0.03" ixy="0" ixz="0" iyy="0.03" iyz="0" izz="0.03" />
       </inertial>
--->
       <visual>
         <origin xyz="0 0 0" rpy="0 0 0" />
@@ -183,6 +175,5 @@
     </joint>
     <link name="${name}_5_link">
-      <xacro:default_inertial/>
-<!--
+      <!--xacro:default_inertial/-->
       <inertial>
         <origin xyz="0 0 0" rpy="0 0 0"/>
@@ -190,5 +181,4 @@
         <inertia ixx="0.03" ixy="0" ixz="0" iyy="0.03" iyz="0" izz="0.03" />
       </inertial>
--->
       <visual>
         <origin xyz="0 0 0" rpy="0 0 0" />
@@ -215,6 +205,5 @@
     </joint>
     <link name="${name}_6_link">
-      <xacro:default_inertial/>
-<!--
+      <!--xacro:default_inertial/-->
       <inertial>
         <origin xyz="0 0 0" rpy="0 0 0"/>
@@ -222,5 +211,4 @@
         <inertia ixx="0.01" ixy="0" ixz="0" iyy="0.01" iyz="0" izz="0.01" />
       </inertial>
--->
       <visual>
         <origin xyz="0 0 0" rpy="0 0 0" />
@@ -234,4 +222,74 @@
         <geometry>
           <mesh filename="package://schunk_description/meshes/lwa4p/arm_6_link.stl" />
+        </geometry>
+      </collision>
+    </link>
+    <!-- joint between arm_6_link and Gripper -->
+    <joint name="${name}_gripper_base" type="fixed">
+      <origin xyz="0 0 0.075" rpy="0 0 0" />
+      <parent link="${name}_6_link" />
+      <child link="${name}_gripper_link" />
+    </joint>
+    <link name="${name}_gripper_link">
+      <xacro:default_inertial/>
+      <visual>
+        <origin xyz="-0.03 0.032 0.007" rpy="1.5708 0 0" />
+        <geometry>
+          <mesh filename="package://schunk_description/meshes/lwa4p/gripper_base.STL" scale="0.001 0.001 0.001" />
+        </geometry>
+        <material name="Schunk/Blue" />
+      </visual>
+      <collision>
+        <origin xyz="-0.03 0.032 0.007" rpy="1.5708 0 0" />
+        <geometry>
+          <mesh filename="package://schunk_description/meshes/lwa4p/gripper_base.STL" scale="0.001 0.001 0.001" />
+        </geometry>
+      </collision>
+    </link>
+    <!-- joint between gripper_base and finger1 -->
+    <joint name="${name}_finger1" type="fixed">
+      <origin xyz="0 -0.015 0.11" rpy="0 0 0" />
+      <parent link="${name}_gripper_link" />
+      <child link="${name}_finger1_link" />
+      <!--axis xyz="0 1 0" />
+      <limit effort="1" velocity="1.26" lower="${-0.01}" upper="${0}" /-->
+    </joint>
+    <link name="${name}_finger1_link">
+      <xacro:default_inertial/>
+      <visual>
+        <origin xyz="0.01 -0.01 0.028" rpy="0 1.5708 1.5708" />
+        <geometry>
+          <mesh filename="package://schunk_description/meshes/lwa4p/finger1.STL" scale="0.001 0.001 0.001" />
+        </geometry>
+        <material name="Schunk/LightGrey" />
+      </visual>
+      <collision>
+        <origin xyz="0.01 -0.01 0.028" rpy="0 1.5708 1.5708" />
+        <geometry>
+          <mesh filename="package://schunk_description/meshes/lwa4p/finger1.STL" scale="0.001 0.001 0.001" />
+        </geometry>
+      </collision>
+    </link>
+    <!-- joint between gripper_base and finger2 -->
+    <joint name="${name}_finger2" type="fixed">
+      <origin xyz="0 0.015 0.11" rpy="0 0 0" />
+      <parent link="${name}_gripper_link" />
+      <child link="${name}_finger2_link" />
+      <!--axis xyz="0 1 0" />
+      <limit effort="1" velocity="1.26" lower="${0}" upper="${0.01}" /-->
+    </joint>
+    <link name="${name}_finger2_link">
+      <xacro:default_inertial/>
+      <visual>
+        <origin xyz="0.01 0.0 0.028" rpy="0 1.5708 1.5708" />
+        <geometry>
+          <mesh filename="package://schunk_description/meshes/lwa4p/finger1.STL" scale="0.001 0.001 0.001" />
+        </geometry>
+        <material name="Schunk/LightGrey" />
+      </visual>
+      <collision>
+        <origin xyz="0.01 0.0 0.028" rpy="0 1.5708 1.5708" />
+        <geometry>
+          <mesh filename="package://schunk_description/meshes/lwa4p/finger1.STL" scale="0.001 0.001 0.001" />
         </geometry>
       </collision>
